File: bread_bug.sch (KiCad schematic (older format))
At the start: 28 parts, among them J1 Eurorack PWR, J2 +12V, J3 -12V, J4 +3.3V, J5 +5V, J6 Rail 1, J7 Rail 1 Jumper, J8 Rail 2 Jumper, J9 Rail 2, SW1 Toggle Switch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

Commit message: Rename to Bread Bug
Parts:
- added J10: GND, Connector_PinHeader_2.54mm:PinHeader_1x02_P2.54mm_Vertical, symbol Connector_Generic:Conn_01x02
- C1, C2, C3, C4, C6, C8: footprint Capacitor_SMD:C_0805_2012Metric -> Capacitor_SMD:C_0805_2012Metric_Pad1.15x1.40mm_HandSolder
- C5, C7: footprint Capacitor_SMD:C_0603_1608Metric -> Capacitor_SMD:C_0805_2012Metric_Pad1.15x1.40mm_HandSolder
- F1: footprint Fuse:Fuse_1206_3216Metric -> Fuse:Fuse_1206_3216Metric_Pad1.42x1.75mm_HandSolder
- FB1, FB2: footprint Inductor_SMD:L_0805_2012Metric -> Inductor_SMD:L_0805_2012Metric_Pad1.15x1.40mm_HandSolder
- L1: footprint Inductor_SMD:L_0603_1608Metric -> Inductor_SMD:L_0805_2012Metric_Pad1.15x1.40mm_HandSolder
Connections:
- net GND: now also J10.1 (Pin_1), J10.2 (Pin_2)
Changed lines of the file:
@@
 F 0 "FB2" V 3526 1850 50  0000 C CNN
 F 1 "100 @ 100MHz" V 3617 1850 50  0000 C CNN
-F 2 "Inductor_SMD:L_0805_2012Metric" V 3730 1850 50  0001 C CNN
+F 2 "Inductor_SMD:L_0805_2012Metric_Pad1.15x1.40mm_HandSolder" V 3730 1850 50  0001 C CNN
 F 3 "~" H 3800 1850 50  0001 C CNN
 	1    3800 1850
@@
 F 0 "FB1" V 3526 1450 50  0000 C CNN
 F 1 "100 @ 100MHz" V 3617 1450 50  0000 C CNN
-F 2 "Inductor_SMD:L_0805_2012Metric" V 3730 1450 50  0001 C CNN
+F 2 "Inductor_SMD:L_0805_2012Metric_Pad1.15x1.40mm_HandSolder" V 3730 1450 50  0001 C CNN
 F 3 "~" H 3800 1450 50  0001 C CNN
 	1    3800 1450
@@
 F 0 "C7" H 2965 3946 50  0000 L CNN
 F 1 "100n" H 2965 3855 50  0000 L CNN
-F 2 "Capacitor_SMD:C_0603_1608Metric" H 2888 3750 50  0001 C CNN
+F 2 "Capacitor_SMD:C_0805_2012Metric_Pad1.15x1.40mm_HandSolder" H 2888 3750 50  0001 C CNN
 F 3 "~" H 2850 3900 50  0001 C CNN
 	1    2850 3900
@@
 F 0 "C1" V 4348 1450 50  0000 C CNN
 F 1 "22u" V 4439 1450 50  0000 C CNN
-F 2 "Capacitor_SMD:C_0805_2012Metric" H 4638 1300 50  0001 C CNN
+F 2 "Capacitor_SMD:C_0805_2012Metric_Pad1.15x1.40mm_HandSolder" H 4638 1300 50  0001 C CNN
 F 3 "~" H 4600 1450 50  0001 C CNN
 	1    4600 1450
@@
 F 0 "C2" V 4348 1850 50  0000 C CNN
 F 1 "22u" V 4439 1850 50  0000 C CNN
-F 2 "Capacitor_SMD:C_0805_2012Metric" H 4638 1700 50  0001 C CNN
+F 2 "Capacitor_SMD:C_0805_2012Metric_Pad1.15x1.40mm_HandSolder" H 4638 1700 50  0001 C CNN
 F 3 "~" H 4600 1850 50  0001 C CNN
 	1    4600 1850
@@
 F 0 "C8" H 3665 3946 50  0000 L CNN
 F 1 "10u" H 3665 3855 50  0000 L CNN
-F 2 "Capacitor_SMD:C_0805_2012Metric" H 3588 3750 50  0001 C CNN
+F 2 "Capacitor_SMD:C_0805_2012Metric_Pad1.15x1.40mm_HandSolder" H 3588 3750 50  0001 C CNN
 F 3 "~" H 3550 3900 50  0001 C CNN
 	1    3550 3900
@@
 F 0 "C6" H 9435 1554 50  0000 R CNN
 F 1 "22u" H 9435 1645 50  0000 R CNN
-F 2 "Capacitor_SMD:C_0805_2012Metric" H 9588 1450 50  0001 C CNN
+F 2 "Capacitor_SMD:C_0805_2012Metric_Pad1.15x1.40mm_HandSolder" H 9588 1450 50  0001 C CNN
 F 3 "~" H 9550 1600 50  0001 C CNN
 	1    9550 1600
@@
 F 0 "C4" H 7585 1554 50  0000 R CNN
 F 1 "10u" H 7585 1645 50  0000 R CNN
-F 2 "Capacitor_SMD:C_0805_2012Metric" H 7738 1450 50  0001 C CNN
+F 2 "Capacitor_SMD:C_0805_2012Metric_Pad1.15x1.40mm_HandSolder" H 7738 1450 50  0001 C CNN
 F 3 "~" H 7700 1600 50  0001 C CNN
 	1    7700 1600
@@
 F 0 "C3" H 7115 1646 50  0000 L CNN
 F 1 "10u" H 7115 1555 50  0000 L CNN
-F 2 "Capacitor_SMD:C_0805_2012Metric" H 7038 1450 50  0001 C CNN
+F 2 "Capacitor_SMD:C_0805_2012Metric_Pad1.15x1.40mm_HandSolder" H 7038 1450 50  0001 C CNN
 F 3 "~" H 7000 1600 50  0001 C CNN
 	1    7000 1600
@@
 F 0 "C5" H 9115 1646 50  0000 L CNN
 F 1 "100n" H 9115 1555 50  0000 L CNN
-F 2 "Capacitor_SMD:C_0603_1608Metric" H 9038 1450 50  0001 C CNN
+F 2 "Capacitor_SMD:C_0805_2012Metric_Pad1.15x1.40mm_HandSolder" H 9038 1450 50  0001 C CNN
 F 3 "~" H 9000 1600 50  0001 C CNN
 	1    9000 1600
@@
 F 0 "L1" V 7540 1450 50  0000 C CNN
 F 1 "10u" V 7449 1450 50  0000 C CNN
-F 2 "Inductor_SMD:L_0603_1608Metric" H 7350 1450 50  0001 C CNN
+F 2 "Inductor_SMD:L_0805_2012Metric_Pad1.15x1.40mm_HandSolder" H 7350 1450 50  0001 C CNN
 F 3 "~" H 7350 1450 50  0001 C CNN
 	1    7350 1450
@@
 F 0 "F1" V 6725 1450 50  0000 C CNN
 F 1 "1A" V 6634 1450 50  0000 C CNN
-F 2 "Fuse:Fuse_1206_3216Metric" H 6550 1250 50  0001 L CNN
+F 2 "Fuse:Fuse_1206_3216Metric_Pad1.42x1.75mm_HandSolder" H 6550 1250 50  0001 L CNN
 F 3 "~" H 6500 1450 50  0001 C CNN
 	1    6500 1450
 	0    -1   -1   0
 $EndComp
+$Comp
+L Connector_Generic:Conn_01x02 J10
+U 1 1 5FAB31DC
+P 6850 5150
+F 0 "J10" H 6930 5142 50  0000 L CNN
+F 1 "GND" H 6930 5051 50  0000 L CNN
+F 2 "Connector_PinHeader_2.54mm:PinHeader_1x02_P2.54mm_Vertical" H 6850 5150 50  0001 C CNN
+F 3 "~" H 6850 5150 50  0001 C CNN
+	1    6850 5150
+	1    0    0    -1
+$EndComp
+Wire Wire Line
+	6450 5150 6650 5150
+Wire Wire Line
+	6650 5150 6650 5250
+Connection ~ 6650 5150
+$Comp
+L power:GND #PWR0109
+U 1 1 5FAB8396
+P 6450 5150
+F 0 "#PWR0109" H 6450 4900 50  0001 C CNN
+F 1 "GND" H 6455 4977 50  0000 C CNN
+F 2 "" H 6450 5150 50  0001 C CNN
+F 3 "" H 6450 5150 50  0001 C CNN
+	1    6450 5150
+	0    1    1    0
+$EndComp
 $EndSCHEMATC
